File: Elproj2.kicad_sch (KiCad schematic)
At the start: 13 parts, among them U1 ${SIM.PARAMS}, U2 ${SIM.PARAMS}

Commit message: Här är kresterna för filtret och förstärkaren, men inget har simulerats än
Other:
- title: Elproj2 -> (none)
Changed lines of the file:
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@@
 	(generator_version "9.0")
 	(paper "A4")
-	(title_block
-		(title "Elproj2")
-	)
 	(text_box "Kretsen för filtret"
 		(exclude_from_sim no)
